File: hardware/TOP/RiseUpTop.brd (EAGLE design)
At the start: 38 x 38 mm, 52 parts, among them SW1 SWITCH.MOM, SW2 SWITCH.MOM, SW5 SWITCH.MOM, U2 NRF52832_MODULE_MDBT42, U4 PCF8523

Commit message: updated TOP board
Parts:
- moved SW5 42.5 mm to (32.0, 3.48)
- moved SW2 27.4 mm to (19.1, 3.43)
- moved SW1 12.2 mm to (6.12, 3.40)
- moved D5 6.87 mm to (11.2, 7.70)
- moved R15 6.56 mm to (20.5, 8.53)
- moved LDO2 6.48 mm to (16.3, 8.48)
- moved C6 6.47 mm to (18.9, 8.51)
- moved C5 6.37 mm to (13.6, 8.51)
- moved D4 6.28 mm to (11.1, 9.19)
- moved R12 5.13 mm to (19.5, 11.0)
- moved C21 4.47 mm to (17.1, 11.6)
- moved CHRG2 4.17 mm to (14.2, 11.6)
- moved C20 4.02 mm to (11.5, 11.6)
- moved R14 2.97 mm to (9.80, 11.7)
- moved R13 2.17 mm to (8.08, 11.6)
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Connections:
- net VBATT renamed VBAT
- removed net N$16: SW1.A1
- removed net N$18: SW1.B1, SW1.B2
- new net SW1: SW1.A1, SW2.A1, SW5.A1
- net GND: now also SW1.B1, SW1.B2, SW2.B1, SW2.B2, SW5.B1, SW5.B2, USB2.S1, USB2.S2, USB2.S3, USB2.S4, USB2.S5, USB2.S6

Commit message: updated top board
Parts:
- removed C10: 300p, LinnesLab-Passives:C0603
- removed C7: 1u, LinnesLab-Passives:C0603
- removed C8, C9: (no value), LinnesLab-Passives:C0603
- removed R9: 10k, LinnesLab-Passives:R0603
- removed SW3, SW4: (no value), LinnesLab-Switches:BUTTON-GULLWING
- added C22, C23: 300p, LinnesLab-Passives:C0603
- added C24: 10u, LinnesLab-Passives:C0805
- added C25, C29: 100n, LinnesLab-Passives:C0603
- added C30, C31: 47p, LinnesLab-Passives:C0603
- added JP2: (no value), LinnesLab-Switches:SMT-JUMPER_2_NO_SILK
- added LED7: RED, LinnesLab-LED:LED-0603
- added LED8: YELLOW, LinnesLab-LED:LED-0603
- added R1, R2: 0, LinnesLab-Passives:R0603
- added R10: 10k, LinnesLab-Passives:R0603
- added R20, R21: 27, LinnesLab-Passives:R0603
- added R22, R23: 1k, LinnesLab-Passives:R0603
- added SW6, SW7: (no value), LinnesLab-Switches:BUTTON-GULLWING
- added U6: FT231XS, LinnesLab-DigitalIC:SSOP20_L
- C11: value 300p -> 1u
- C12: value 10u -> (none); device LinnesLab-Passives:C0805 -> LinnesLab-Passives:C0603
- C14: value 100n -> (none)
- R3: value 1k -> 10k
- R5: value 10k -> 1k
- moved R3 58.8 mm to (-5.89, -12.0), turned to 0 degrees
- moved R8 43.4 mm to (-5.89, -14.7), turned to 0 degrees
- moved XTAL3 32.0 mm to (3.33, -4.75)
- moved U4 31.9 mm to (7.90, -6.22)
- moved C2 31.5 mm to (9.70, -2.62)
- moved R5 30.2 mm to (16.8, 30.0), turned to 180 degrees
- moved D1 29.5 mm to (18.5, 24.9)
- moved CORTEX1 23.8 mm to (17.8, 33.4)
- moved LED4 23.0 mm to (20.5, 29.8)
- moved LED3 22.9 mm to (20.4, 27.7)
- moved R4 22.8 mm to (17.0, 27.8)
- moved C14 19.5 mm to (30.9, 15.4), turned to 0 degrees
- moved C11 12.9 mm to (24.8, 26.6), turned to 270 degrees
- moved C12 7.20 mm to (26.2, 15.5)
- moved U2 0.87 mm to (31.8, 29.5)
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Connections:
- removed net N$10: LED4.A, R4.1
- removed net N$12: C7.1, L2.2, U2.9
- removed net N$4 (its old number): C8.2, U2.13, XTAL2.P$1
- removed net N$6 (its old number): C9.1, U2.14, XTAL2.P$2
- removed net N$9: LED3.A, R3.1
- removed net RXD: U2.21
- removed net TXD: U2.19
- new net !CTS: JP2.2, U6.9
- new net FT3V3: U6.13
- new net N$16: C12.2, U2.13, XTAL2.P$1
- new net N$18: C14.1, U2.14, XTAL2.P$2
- new net N$21: LED3.A, R4.1
- new net N$22: LED4.A, R5.1
- new net N$24: C11.1, L2.2, U2.9
- new net N$30: R20.2, U6.12
- new net N$31: R21.2, U6.11
- new net N$32: LED7.C, R22.2
- new net N$33: LED8.C, R23.2
- new net RXD.FT: R2.1, U6.4
- new net RXD.NRF: R1.2, U2.21
- new net RXLED: R22.1, U6.17
- new net TXD.FT: R1.1, U6.20
- new net TXD.NRF: R2.2, U2.19
- new net TXLED: R23.1, U6.10
- net 3.3V: now also C24.2, C29.2, LED7.A, LED8.A, R10.2, R3.2, U6.14, U6.3; no longer C12.2, R5.2, R9.2
- net DFU: now also SW6.3; no longer SW3.3
- net DTR: now also C25.1, U6.1; no longer C14.1
- net GND: now also C14.2, C22.2, C23.2, C24.1, C29.1, C30.2, C31.1, JP2.1, SW6.1, SW7.3, U6.16, U6.6; no longer C10.2, C7.2, C8.1, C9.2, SW3.1, SW4.3
- net LED1: now also R4.2; no longer R3.2
- net LED2: now also R5.2; no longer R4.2
- net P0.09/NFC1: now also C23.1; no longer C11.1
- net P0.10/NFC2: now also C22.1; no longer C10.1
- net RESET: now also C25.2, R10.1, SW7.1; no longer C14.2, R5.1, SW4.1
- net SDA: now also R3.1; no longer R9.1
- net USB+: now also C30.1, R21.1
- net USB-: now also C31.2, R20.1
- net V_USB: now also U6.15

Commit message: almost completed Top board
Parts:
- moved R2 45.6 mm to (35.2, 12.4)
- moved R8 45.1 mm to (31.8, 10.2)
- moved R3 42.9 mm to (31.9, 8.23)
- moved R1 41.3 mm to (31.8, 12.4)
- moved U4 25.2 mm to (26.5, 10.8)
- moved XTAL3 13.9 mm to (13.2, 5.00)
- moved C2 6.10 mm to (12.5, 2.79)
- moved R21 1.35 mm to (2.82, 34.5)
- moved R23 0.56 mm to (5.84, 18.4)
- moved R22 0.40 mm to (5.82, 20.3)
- moved R20 0.38 mm to (2.77, 36.4)
- moved LED7 0.33 mm to (5.54, 23.9)
- moved LED8 0.29 mm to (5.64, 22.0)
- moved C29 0.27 mm to (2.31, 25.3)
- moved JP2 0.25 mm to (1.80, 31.2)
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
Commit message: updated top from Take 2
Parts:
- added J1: (no value), LinnesLab-Connectors:1X07
- moved CORTEX1 6.05 mm to (12.4, 36.1)
- moved R21 3.89 mm to (2.03, 30.7)
- moved R20 3.49 mm to (2.13, 33.0)
- moved JP2 3.48 mm to (1.98, 27.8)
- moved U6 1.31 mm to (7.01, 29.2)
Connections:
- net CHRG.STAT renamed D27/CHRG.STATUS
- removed net BATT: R13.1, R14.2
- removed net SD.CS: SD2.2
- new net A4/BATT: R13.1, R14.2, U2.5
- new net D27/CHRG.STATU: U2.4
- new net D7/SD.CS: SD2.2, U2.20

Commit message: Updates July2nd
Parts:
- added GPS.PWR: MIC5504, LinnesLab-Power:SOT23-5
Connections:
- new net D2/GPS.PWR: GPS.PWR.3, U2.15
Changed lines of the file:
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@@
 <attribute name="VALUE" x="3.73" y="30.968" size="0.6096" layer="27" font="vector" ratio="20"/>
+</element>
+<element name="GPS.PWR" library="LinnesLab-Power" package="SOT23-5" value="MIC5504" x="35.5346" y="18.4658" smashed="yes">
+<attribute name="NAME" x="33.6296" y="18.4658" size="0.6096" layer="25" ratio="20" rot="R90" align="bottom-center"/>
+<attribute name="VALUE" x="38.0746" y="18.4658" size="0.6096" layer="27" ratio="20" rot="R90" align="bottom-center"/>
 </element>
 </elements>
@@
 <wire x1="31.2966" y1="6.451" x2="33.15" y2="21.8394" width="0" layer="19" extent="1-16"/>
 </signal>
+<signal name="D2/GPS.PWR">
+<contactref element="U2" pad="15"/>
+<contactref element="GPS.PWR" pad="3"/>
+<wire x1="36.4846" y1="17.1657" x2="29.65" y2="21.8394" width="0" layer="19" extent="1-1"/>
+</signal>
 </signals>

Commit message: Updates end of July2nd, Start Take 03
Connections:
- removed net CD1: SD2.CD1
- removed net CS.OLED: U3.13
- removed net DC.OLED: U3.15
- removed net RESET.OLED: U3.14
- removed net SW1: SW1.A1, SW2.A1, SW5.A1
- new net A6/TIA: U2.7
- new net A7/PPG: U2.8
- new net D11/SW1: SW1.A1, U2.25
- new net D15/SW2: SW2.A1, U2.29
- new net D16/CS.OLED: U2.30, U3.13
- new net D16/SW3: SW5.A1
- new net D29/LED.CTRL: U2.6
- new net D3/RESET.OLED: U2.16, U3.14
- new net D4/DC.OLED: U2.17, U3.15
- new net D5/CD1: SD2.CD1, U2.18
Changed lines of the file:
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@@
 <wire x1="31.6966" y1="11.951" x2="36.35" y2="25.3894" width="0" layer="19" extent="1-16"/>
-</signal>
-<signal name="DC.OLED">
-<contactref element="U3" pad="15"/>
-</signal>
-<signal name="RESET.OLED">
-<contactref element="U3" pad="14"/>
 </signal>
 <signal name="N$1">
@@
 <wire x1="26.8714" y1="19.882" x2="26.8732" y2="25.415" width="0" layer="19" extent="1-1"/>
 </signal>
-<signal name="CS.OLED">
-<contactref element="U3" pad="13"/>
-</signal>
 <signal name="CD2">
 <contactref element="SD2" pad="CD2"/>
-</signal>
-<signal name="CD1">
-<contactref element="SD2" pad="CD1"/>
 </signal>
 <signal name="N$17">
@@
 <wire x1="12.326" y1="7.6962" x2="12.2498" y2="9.1948" width="0" layer="19" extent="1-1"/>
 </signal>
-<signal name="SW1">
-<contactref element="SW1" pad="A1"/>
-<contactref element="SW2" pad="A1"/>
-<contactref element="SW5" pad="A1"/>
-<wire x1="15.1512" y1="1.179" x2="27.9782" y2="1.2298" width="0" layer="19" extent="1-1"/>
-<wire x1="2.1464" y1="1.1536" x2="15.1512" y2="1.179" width="0" layer="19" extent="1-1"/>
-</signal>
 <signal name="N$30">
 <contactref element="R20" pad="2"/>
@@
 <wire x1="36.4846" y1="17.1657" x2="29.65" y2="21.8394" width="0" layer="19" extent="1-1"/>
 </signal>
+<signal name="D5/CD1">
+<contactref element="U2" pad="18"/>
+<contactref element="SD2" pad="CD1"/>
+<wire x1="21.4966" y1="12.351" x2="31.75" y2="21.8394" width="0" layer="19" extent="1-16"/>
+</signal>
+<signal name="D11/SW1">
+<contactref element="U2" pad="25"/>
+<contactref element="SW1" pad="A1"/>
+<wire x1="2.1464" y1="1.1536" x2="36.35" y2="23.2894" width="0" layer="19" extent="1-1"/>
+</signal>
+<signal name="D15/SW2">
+<contactref element="U2" pad="29"/>
+<contactref element="SW2" pad="A1"/>
+<wire x1="15.1512" y1="1.179" x2="36.35" y2="26.0894" width="0" layer="19" extent="1-1"/>
+</signal>
+<signal name="D16/SW3">
+<contactref element="SW5" pad="A1"/>
+</signal>
+<signal name="D16/CS.OLED">
+<contactref element="U2" pad="30"/>
+<contactref element="U3" pad="13"/>
+<wire x1="17.0714" y1="19.882" x2="36.35" y2="26.7894" width="0" layer="19" extent="1-1"/>
+</signal>
+<signal name="D3/RESET.OLED">
+<contactref element="U2" pad="16"/>
+<contactref element="U3" pad="14"/>
+<wire x1="17.7714" y1="19.882" x2="30.35" y2="21.8394" width="0" layer="19" extent="1-1"/>
+</signal>
+<signal name="D4/DC.OLED">
+<contactref element="U2" pad="17"/>
+<contactref element="U3" pad="15"/>
+<wire x1="18.4714" y1="19.882" x2="31.05" y2="21.8394" width="0" layer="19" extent="1-1"/>
+</signal>
+<signal name="D29/LED.CTRL">
+<contactref element="U2" pad="6"/>
+</signal>
+<signal name="A6/TIA">
+<contactref element="U2" pad="7"/>
+</signal>
+<signal name="A7/PPG">
+<contactref element="U2" pad="8"/>
+</signal>
 </signals>
