File: hardware/TOP/RiseUpTop.sch (EAGLE design)
At the start: 52 parts, among them SW1 SWITCH.MOM, SW2 SWITCH.MOM, SW5 SWITCH.MOM, U2 NRF52832_MODULE_MDBT42, U4 PCF8523

Commit message: updated TOP board
Connections:
- removed net N$16: SW1.1
- removed net N$18: SW1.3, SW1.4
- removed net VBATT: U4.VBAT
- new net SW1: SW1.1, SW2.1, SW5.1
- net GND: now also SW1.3, SW1.4, SW2.3, SW2.4, SW5.3, SW5.4, USB2.SHIELD
Other:
- note added: "Digital Outputs CS. OLED RESET.OLED DC.OLED [SPI] [I2C] - Real-time clock SD.CS (Optional) Card detect 1 and 2 Digital inputs 3x buttons Charge Status Analog inputs Battery monitor Analog Outputs Data to send to bottom board 3.3V GND I2C TIA 2-3x GPIO PPG (Pulse Sensor Circuit Output)"
- note removed: "Additional notes for advanced users only"
- note removed: "Connect MISO, MOSI, and SCK to appropriate pins on microcontroller. Those are SPI pins and are generally prespecified. You have more flexibility with the SD.CS pin."
- note removed: "PIN_DFU / P0.20: If this pin is detected to be at GND level at startup, the board will enter a special serial bootloader mode and will not execute any user code, going straight into bootloader mode. If you wish to use this pin as a standard GPIO, make sure that it is pulled high with a pullup resistor so that your code will execute normally when the MCU starts up. FRST/P0.22: Setting this pin to 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"
- note removed: "SPECIAL / PORT / PIN ON PACKAGE / GPIO(D_or_A) / Comments Factory Reset / P0.22 / pin38 / DO NOT USE FOR ANY GPIO SWDIO / none / pin37 / reserved-not available for general GPIO SWCLK / none / pin36 / reserved-not available for general GPIO RESET / P0.21 / pin35 / reserved-not available for general GPIO DFU / P0.20 / pin34 / reserved-not available for general GPIO LED2 / P0.19 / pin33 / reserved f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"
- note removed: "SPECIAL / PORT / PIN ON PACKAGE / GPIO(D_or_A) / Comments SDA / P0.25 / pin2 / D25 SCL / P0.26 / pin3 / D26 none / P0.27 / pin4 / D27 none / P0.28 / pin5 / D28_or_A4 / (low drive, low frequency IO) none / P0.29 / pin6 / D29_or_A5 / (low drive, low frequency IO) none / P0.30 / pin7 / D30_or_A6 none / P0.31 / pin8 / D31_or_A7 / (used for battery level monitoring on Adafruit boards)"
- note removed: "SPECIAL / PORT / PIN ON PACKAGE / GPIO(D_or_A) / Comments none / P0.02 / pin15 / D2_or_A0 none / P0.03 / pin16 / D3_or_A1 none / P0.04 / pin17 / D4_or_A2 none / P0.05 / pin18 / D5_or_A3 TXD / P0.06 / pin19 / D6 / but reserved for Serial communication and programming none / P0.07 / pin20 / D7 RXD / P0.08 / pin21 / D8 / but reserved for Serial communication and programming NFC1 / P0.09 / pin22 / D9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"
- note removed: "Some pins are noted as reserved and not available for general GPIO (unless you are an adavanced user) I2C, SPI, and SWD pins can be repurposed if you know what you are doing For Milestones, avoid repurposing NFC pins. For P0.19 (LED2), Adafruit's Bluetooth Low Energy libraries use this pin to indicated successful pairing. The LED blinks when the device is doing some Bluetooth process and stays li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"
- moved on the sheet: C13, C14, C15, C16, C17, C18, C19, C2, C20, C21, C5, C6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

Commit message: updated top board
Parts:
- removed C10: 300p, LinnesLab-Passives:CAPACITOR0603
- removed C7: 1u, LinnesLab-Passives:CAPACITOR0603
- removed C8, C9: (no value), LinnesLab-Passives:CAPACITOR0603
- removed R9: 10k, LinnesLab-Passives:RESISTOR0603
- removed SW3, SW4: (no value), LinnesLab-Switches:SPST-PTS830GG140-COPY.1-3
- added C22, C23: 300p, LinnesLab-Passives:CAPACITOR0603
- added C24: 10u, LinnesLab-Passives:CAPACITOR0805
- added C25, C29: 100n, LinnesLab-Passives:CAPACITOR0603
- added C30, C31: 47p, LinnesLab-Passives:CAPACITOR0603
- added JP2: (no value), LinnesLab-Switches:JUMPER-SMT_2_NO_SILK
- added LED7: RED, LinnesLab-LED:LED0603
- added LED8: YELLOW, LinnesLab-LED:LED0603
- added R1, R2: 0, LinnesLab-Passives:RESISTOR0603
- added R10: 10k, LinnesLab-Passives:RESISTOR0603
- added R20, R21: 27, LinnesLab-Passives:RESISTOR0603
- added R22, R23: 1k, LinnesLab-Passives:RESISTOR0603
- added SW6, SW7: (no value), LinnesLab-Switches:SPST-PTS830GG140-COPY.1-3
- added U6: FT231XS, LinnesLab-DigitalIC:FT231XS
- C11: value 300p -> 1u
- C12: value 10u -> (none); device LinnesLab-Passives:CAPACITOR0805 -> LinnesLab-Passives:CAPACITOR0603
- C14: value 100n -> (none)
- R3: value 1k -> 10k
- R5: value 10k -> 1k
Connections:
- removed net N$10: LED4.A, R4.1
- removed net N$12: C7.1, L2.2, U2.DEC4
- removed net N$4 (its old number): C8.2, U2.P0.00/XL1, XTAL2.1
- removed net N$6 (its old number): C9.1, U2.P0.01/XL2, XTAL2.2
- removed net N$9: LED3.A, R3.1
- removed net RXD: U2.P0.08
- removed net TXD: U2.P0.06
- new net !CTS: JP2.2, U6.!CTS
- new net FT3V3: U6.3V3OUT
- new net N$16: C12.2, U2.P0.00/XL1, XTAL2.1
- new net N$18: C14.1, U2.P0.01/XL2, XTAL2.2
- new net N$21: LED3.A, R4.1
- new net N$22: LED4.A, R5.1
- new net N$24: C11.1, L2.2, U2.DEC4
- new net N$30: R20.2, U6.USBDM
- new net N$31: R21.2, U6.USBDP
- new net N$32: LED7.C, R22.2
- new net N$33: LED8.C, R23.2
- new net RXD.FT: R2.1, U6.RXD
- new net RXD.NRF: R1.2, U2.P0.08
- new net RXLED: R22.1, U6.CBUS1
- new net TXD.FT: R1.1, U6.TXD
- new net TXD.NRF: R2.2, U2.P0.06
- new net TXLED: R23.1, U6.CBUS2
- net 3.3V: now also C24.2, C29.2, LED7.A, LED8.A, R10.2, R3.2, U6.!RESET, U6.VCCIO; no longer C12.2, R5.2, R9.2
- net DFU: now also SW6.B; no longer SW3.B
- net DTR: now also C25.1, U6.!DTR; no longer C14.1
- net GND: now also C14.2, C22.2, C23.2, C24.1, C29.1, C30.2, C31.1, JP2.1, SW6.A, SW7.B, U6.GND@16, U6.GND@6; no longer C10.2, C7.2, C8.1, C9.2, SW3.A, SW4.B
- net LED1: now also R4.2; no longer R3.2
- net LED2: now also R5.2; no longer R4.2
- net P0.09/NFC1: now also C23.1; no longer C11.1
- net P0.10/NFC2: now also C22.1; no longer C10.1
- net RESET: now also C25.2, R10.1, SW7.A; no longer C14.2, R5.1, SW4.A
- net SDA: now also R3.1; no longer R9.1
- net USB+: now also C30.1, R21.1
- net USB-: now also C31.2, R20.1
- net V_USB: now also U6.VCC
Other:
- note added: "Additional notes for advanced users only"
- note added: "I don't remember if CTS needs to be grounded or left floating so here's a jumper to ground so it can be configued either way dynamically."
- note added: "Make sure the resistors are next to each other on the board"
- note added: "PIN_DFU / P0.20: If this pin is detected to be at GND level at startup, the board will enter a special serial bootloader mode and will not execute any user code, going straight into bootloader mode. If you wish to use this pin as a standard GPIO, make sure that it is pulled high with a pullup resistor so that your code will execute normally when the MCU starts up. FRST/P0.22: Setting this pin to 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"
- note added: "SPECIAL / PORT / PIN ON PACKAGE / GPIO(D_or_A) / Comments Factory Reset / P0.22 / pin38 / DO NOT USE FOR ANY GPIO SWDIO / none / pin37 / reserved-not available for general GPIO SWCLK / none / pin36 / reserved-not available for general GPIO RESET / P0.21 / pin35 / reserved-not available for general GPIO DFU / P0.20 / pin34 / reserved-not available for general GPIO LED2 / P0.19 / pin33 / reserved f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"
- note added: "SPECIAL / PORT / PIN ON PACKAGE / GPIO(D_or_A) / Comments SDA / P0.25 / pin2 / D25 SCL / P0.26 / pin3 / D26 none / P0.27 / pin4 / D27 none / P0.28 / pin5 / D28_or_A4 / (low drive, low frequency IO) none / P0.29 / pin6 / D29_or_A5 / (low drive, low frequency IO) none / P0.30 / pin7 / D30_or_A6 none / P0.31 / pin8 / D31_or_A7 / (used for battery level monitoring on Adafruit boards)"
- note added: "SPECIAL / PORT / PIN ON PACKAGE / GPIO(D_or_A) / Comments none / P0.02 / pin15 / D2_or_A0 none / P0.03 / pin16 / D3_or_A1 none / P0.04 / pin17 / D4_or_A2 none / P0.05 / pin18 / D5_or_A3 TXD / P0.06 / pin19 / D6 / but reserved for Serial communication and programming none / P0.07 / pin20 / D7 RXD / P0.08 / pin21 / D8 / but reserved for Serial communication and programming NFC1 / P0.09 / pin22 / D9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"
- note added: "Some pins are noted as reserved and not available for general GPIO (unless you are an adavanced user) I2C, SPI, and SWD pins can be repurposed if you know what you are doing For Milestones, avoid repurposing NFC pins. For P0.19 (LED2), Adafruit's Bluetooth Low Energy libraries use this pin to indicated successful pairing. The LED blinks when the device is doing some Bluetooth process and stays li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"
- note added: "TXD goes to RX on the other device RXD goes to TX on the other device"
- note removed: "RTC"
- moved on the sheet: C11, C12, C14, C2, CORTEX1, D1, L2, LED3, LED4, R3, R4, R5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

Commit message: almost completed Top board
Other:
- note added: "FTDI Serial-to-USB Converter"
- note added: "Notes"
- moved on the sheet: C11, C12, C14, C22, C23, C24, C29, C30, C31, JP2, L2, LED3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

Commit message: updated top from Take 2
Parts:
- added J1: (no value), LinnesLab-Connectors:CONN_07
Connections:
- net CHRG.STAT renamed D27/CHRG.STATUS
- removed net BATT: R13.1, R14.2
- removed net SD.CS: SD2.CS
- new net A4/BATT: R13.1, R14.2, U2.P0.28/AIN4
- new net D27/CHRG.STATU: U2.P0.27
- new net D7/SD.CS: SD2.CS, U2.P0.07
Other:
- note added: "Digital Output"
- note added: "Notes: Might have to change the connector Need to put more space at the left of the microcontroller"
Changed lines of the file:
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@@
 <part name="SUPPLY1" library="LinnesLab-Symbols" deviceset="3.3V" device=""/>
 <part name="SUPPLY3" library="LinnesLab-Symbols" deviceset="3.3V" device=""/>
+<part name="J1" library="LinnesLab-Connectors" deviceset="CONN_07" device=""/>
 </parts>
 <sheets>
@@
 <wire x1="238.76" y1="317.5" x2="238.76" y2="139.7" width="1.27" layer="94" style="longdash"/>
 <text x="83.82" y="116.84" size="2.54" layer="97" font="vector">Notes</text>
+<text x="96.52" y="-81.28" size="1.27" layer="96">Digital Output</text>
+<text x="-25.4" y="104.14" size="1.27" layer="97">Notes:
+Might have to change the connector
+Need to put more space at the left of the microcontroller</text>
 </plain>
 <instances>
@@
 <instance part="SUPPLY3" gate="G$1" x="63.5" y="294.64" smashed="yes">
 <attribute name="VALUE" x="63.5" y="297.434" size="1.778" layer="96" align="bottom-center"/>
+</instance>
+<instance part="J1" gate="G$1" x="-7.62" y="86.36" smashed="yes">
+<attribute name="VALUE" x="-12.7" y="76.454" size="1.778" layer="96" font="vector"/>
+<attribute name="NAME" x="0" y="89.408" size="1.778" layer="95" font="vector"/>
 </instance>
 </instances>
@@
 </segment>
 </net>
-<net name="SD.CS" class="0">
-<segment>
-<wire x1="198.12" y1="-50.8" x2="203.2" y2="-50.8" width="0.1524" layer="91"/>
-<label x="198.12" y="-50.8" size="1.27" layer="95" rot="R180" xref="yes"/>
-<pinref part="SD2" gate="G$1" pin="CS"/>
-</segment>
-</net>
 <net name="N$17" class="0">
 <segment>
@@
 </segment>
 </net>
-<net name="CHRG.STAT" class="0">
+<net name="D27/CHRG.STATUS" class="0">
 <segment>
 <pinref part="R12" gate="G$1" pin="1"/>
@@
 <junction x="261.62" y="241.3"/>
 <label x="248.92" y="241.3" size="1.27" layer="95" ratio="15" rot="R180" xref="yes"/>
-</segment>
-</net>
-<net name="BATT" class="0">
-<segment>
-<pinref part="R13" gate="G$1" pin="1"/>
-<pinref part="R14" gate="G$1" pin="2"/>
-<wire x1="152.4" y1="-50.8" x2="152.4" y2="-45.72" width="0.1524" layer="91"/>
-<label x="152.4" y="-48.26" size="1.27" layer="95" xref="yes"/>
 </segment>
 </net>
@@
 </segment>
 </net>
+<net name="D27/CHRG.STATU" class="0">
+<segment>
+<pinref part="U2" gate="G$1" pin="P0.27"/>
+<wire x1="109.22" y1="259.08" x2="106.68" y2="259.08" width="0.1524" layer="91"/>
+<label x="106.68" y="259.08" size="1.27" layer="95" rot="R180" xref="yes"/>
+</segment>
+</net>
+<net name="A4/BATT" class="0">
+<segment>
+<pinref part="U2" gate="G$1" pin="P0.28/AIN4"/>
+<wire x1="109.22" y1="256.54" x2="106.68" y2="256.54" width="0.1524" layer="91"/>
+<label x="106.68" y="256.54" size="1.27" layer="95" rot="R180" xref="yes"/>
+</segment>
+<segment>
+<pinref part="R13" gate="G$1" pin="1"/>
+<pinref part="R14" gate="G$1" pin="2"/>
+<wire x1="152.4" y1="-50.8" x2="152.4" y2="-45.72" width="0.1524" layer="91"/>
+<label x="152.4" y="-48.26" size="1.27" layer="95" xref="yes"/>
+</segment>
+</net>
+<net name="D7/SD.CS" class="0">
+<segment>
+<pinref part="U2" gate="G$1" pin="P0.07"/>
+<wire x1="137.16" y1="226.06" x2="137.16" y2="223.52" width="0.1524" layer="91"/>
+<label x="137.16" y="223.52" size="1.27" layer="95" rot="R270" xref="yes"/>
+</segment>
+<segment>
+<wire x1="198.12" y1="-50.8" x2="203.2" y2="-50.8" width="0.1524" layer="91"/>
+<label x="198.12" y="-50.8" size="1.27" layer="95" rot="R180" xref="yes"/>
+<pinref part="SD2" gate="G$1" pin="CS"/>
+</segment>
+</net>

Commit message: Updates July2nd
Parts:
- added GPS.PWR: MIC5504, LinnesLab-Power:MIC5504
Connections:
- new net D2/GPS.PWR: GPS.PWR.EN, U2.P0.02/AIN0
Changed lines of the file:
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@@
 <part name="SUPPLY3" library="LinnesLab-Symbols" deviceset="3.3V" device=""/>
 <part name="J1" library="LinnesLab-Connectors" deviceset="CONN_07" device=""/>
+<part name="GPS.PWR" library="LinnesLab-Power" deviceset="MIC5504" device=""/>
 </parts>
 <sheets>
@@
 <attribute name="NAME" x="0" y="89.408" size="1.778" layer="95" font="vector"/>
 </instance>
+<instance part="GPS.PWR" gate="G$1" x="154.94" y="-15.24" smashed="yes">
+<attribute name="NAME" x="147.32" y="-6.35" size="1.778" layer="95"/>
+<attribute name="VALUE" x="147.32" y="-25.4" size="1.778" layer="96"/>
+</instance>
 </instances>
 <busses>
@@
 </segment>
 </net>
+<net name="D2/GPS.PWR" class="0">
+<segment>
+<pinref part="U2" gate="G$1" pin="P0.02/AIN0"/>
+<wire x1="124.46" y1="226.06" x2="124.46" y2="223.52" width="0.1524" layer="91"/>
+<label x="124.46" y="223.52" size="1.27" layer="95" rot="R270" xref="yes"/>
+</segment>
+<segment>
+<pinref part="GPS.PWR" gate="G$1" pin="EN"/>
+<wire x1="144.78" y1="-20.32" x2="142.24" y2="-20.32" width="0.1524" layer="91"/>
+<label x="142.24" y="-20.32" size="1.778" layer="95" rot="R180" xref="yes"/>
+</segment>
+</net>

Commit message: Updates end of July2nd, Start Take 03
Connections:
- removed net CD1: SD2.CARD_DETECT
- removed net CS.OLED: U3./CS
- removed net DC.OLED: U3.DC/I2C_SA0
- removed net RESET.OLED: U3./RES
- removed net SW1: SW1.1, SW2.1, SW5.1
- new net A6/TIA: U2.P0.30/AIN6
- new net A7/PPG: U2.P0.31/AIN7
- new net D11/SW1: SW1.1, U2.P0.11
- new net D15/SW2: SW2.1, U2.P0.15
- new net D16/CS.OLED: U2.P0.16, U3./CS
- new net D16/SW3: SW5.1
- new net D29/LED.CTRL: U2.P0.29/AIN5
- new net D3/RESET.OLED: U2.P0.03/AIN1, U3./RES
- new net D4/DC.OLED: U2.P0.04/AIN2, U3.DC/I2C_SA0
- new net D5/CD1: SD2.CARD_DETECT, U2.P0.05/AIN3
Other:
- note added: "Find a pin to connect the third button if necessary"
- note added: "Make sure the resistors are next to each other on board"
- note added: "Power management D27/CHRG.STATUS (input to micro) A4/BATT (Input) PPG Circuit D29/LED.CTRL (ouput) A6/TIA (Input) A7/PPG (Input) OLED Pins D3/RESET.OLED (ouput) D4/DC.OLED (ouput) D16/CS.OLED (ouput) SD Card Pins D5/CD1 (Input) D7/SD.CS (ouput) Buttons Inputs D11/SW1 (Input) D15/SW2 (Input) NEED to add SW3"
- note removed: "Make sure the resistors are next to each other on the board"
Changed lines of the file:
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@@
 <text x="45.72" y="213.36" size="1.524" layer="97" font="vector" ratio="15">Additional notes for
 advanced users only</text>
-<text x="345.44" y="259.08" size="1.27" layer="91" ratio="15">Make sure the resistors are next to each other on the board </text>
 <text x="337.82" y="-83.82" size="1.27" layer="97">I2C Address = 0x68h</text>
 <text x="294.64" y="-83.82" size="1.27" layer="97">Back-up
@@
 Might have to change the connector
 Need to put more space at the left of the microcontroller</text>
+<text x="347.98" y="259.08" size="1.27" layer="97">Make sure the resistors are next to each other on board</text>
+<text x="350.52" y="-35.56" size="1.27" layer="97">Find a pin to connect the third button if necessary</text>
+<text x="421.64" y="-22.86" size="1.778" layer="97">Power management
+D27/CHRG.STATUS (input to micro)
+A4/BATT (Input)
+PPG Circuit
+D29/LED.CTRL (ouput)
+A6/TIA (Input)
+A7/PPG (Input)
+OLED Pins
+D3/RESET.OLED (ouput)
+D4/DC.OLED (ouput)
+D16/CS.OLED (ouput)
+SD Card Pins
+D5/CD1 (Input)
+D7/SD.CS (ouput)
+Buttons Inputs
+D11/SW1 (Input)
+D15/SW2 (Input)
+NEED to add SW3
+</text>
 </plain>
 <instances>
@@
 <net name="SCK" class="0">
 <segment>
-<label x="299.72" y="71.12" size="1.778" layer="95"/>
 <pinref part="U3" gate="G$1" pin="D0/SPI_SCLK/I2C_SCK"/>
-<wire x1="325.12" y1="71.12" x2="299.72" y2="71.12" width="0.1524" layer="91"/>
+<wire x1="325.12" y1="71.12" x2="322.58" y2="71.12" width="0.1524" layer="91"/>
+<label x="322.58" y="71.12" size="1.27" layer="95" rot="R180" xref="yes"/>
 </segment>
 <segment>
@@
 <net name="MOSI" class="0">
 <segment>
-<label x="299.72" y="68.58" size="1.778" layer="95"/>
 <pinref part="U3" gate="G$1" pin="D1/SPI_SDIN/I2C_SDA"/>
-<wire x1="325.12" y1="68.58" x2="299.72" y2="68.58" width="0.1524" layer="91"/>
+<wire x1="325.12" y1="68.58" x2="322.58" y2="68.58" width="0.1524" layer="91"/>
+<label x="322.58" y="68.58" size="1.27" layer="95" rot="R180" xref="yes"/>
 </segment>
 <segment>
@@
 <pinref part="U2" gate="G$1" pin="P0.14"/>
 <label x="157.48" y="246.38" size="1.27" layer="95" xref="yes"/>
-</segment>
-</net>
-<net name="DC.OLED" class="0">
-<segment>
-<label x="299.72" y="78.74" size="1.778" layer="95"/>
-<pinref part="U3" gate="G$1" pin="DC/I2C_SA0"/>
-<wire x1="325.12" y1="78.74" x2="299.72" y2="78.74" width="0.1524" layer="91"/>
-</segment>
-</net>
-<net name="RESET.OLED" class="0">
-<segment>
-<label x="299.72" y="81.28" size="1.778" layer="95"/>
-<pinref part="U3" gate="G$1" pin="/RES"/>
-<wire x1="325.12" y1="81.28" x2="299.72" y2="81.28" width="0.1524" layer="91"/>
 </segment>
 </net>
@@
 </segment>
 </net>
-<net name="CS.OLED" class="0">
-<segment>
-<label x="299.72" y="83.82" size="1.778" layer="95"/>
-<pinref part="U3" gate="G$1" pin="/CS"/>
-<wire x1="325.12" y1="83.82" x2="299.72" y2="83.82" width="0.1524" layer="91"/>
-</segment>
-</net>
 <net name="CD2" class="0">
 <segment>
@@
 <label x="198.12" y="-35.56" size="1.27" layer="95" rot="R180" xref="yes"/>
 <pinref part="SD2" gate="G$1" pin="CARD_DETECT1"/>
-</segment>
-</net>
-<net name="CD1" class="0">
-<segment>
-<wire x1="198.12" y1="-33.02" x2="203.2" y2="-33.02" width="0.1524" layer="91"/>
-<label x="198.12" y="-33.02" size="1.27" layer="95" rot="R180" xref="yes"/>
-<pinref part="SD2" gate="G$1" pin="CARD_DETECT"/>
 </segment>
 </net>
@@
 </segment>
 </net>
-<net name="SW1" class="0">
-<segment>
-<pinref part="SW1" gate="G$1" pin="1"/>
-<label x="287.02" y="-20.32" size="1.27" layer="95" ratio="15" rot="R180" xref="yes"/>
-<wire x1="287.02" y1="-20.32" x2="292.1" y2="-20.32" width="0.1524" layer="91"/>
-</segment>
-<segment>
-<pinref part="SW2" gate="G$1" pin="1"/>
-<label x="320.04" y="-20.32" size="1.27" layer="95" ratio="15" rot="R180" xref="yes"/>
-<wire x1="320.04" y1="-20.32" x2="325.12" y2="-20.32" width="0.1524" layer="91"/>
-</segment>
-<segment>
-<pinref part="SW5" gate="G$1" pin="1"/>
-<label x="353.06" y="-20.32" size="1.27" layer="95" ratio="15" rot="R180" xref="yes"/>
-<wire x1="353.06" y1="-20.32" x2="358.14" y2="-20.32" width="0.1524" layer="91"/>
-</segment>
-</net>
 <net name="N$30" class="0">
 <segment>
@@
 </segment>
 </net>
+<net name="D5/CD1" class="0">
+<segment>
+<pinref part="U2" gate="G$1" pin="P0.05/AIN3"/>
+<wire x1="132.08" y1="226.06" x2="132.08" y2="223.52" width="0.1524" layer="91"/>
+<label x="132.08" y="223.52" size="1.27" layer="95" rot="R270" xref="yes"/>
+</segment>
+<segment>
+<wire x1="198.12" y1="-33.02" x2="203.2" y2="-33.02" width="0.1524" layer="91"/>
+<label x="198.12" y="-33.02" size="1.27" layer="95" rot="R180" xref="yes"/>
+<pinref part="SD2" gate="G$1" pin="CARD_DETECT"/>
+</segment>
+</net>
+<net name="D11/SW1" class="0">
+<segment>
+<pinref part="U2" gate="G$1" pin="P0.11"/>
+<wire x1="154.94" y1="238.76" x2="157.48" y2="238.76" width="0.1524" layer="91"/>
+<label x="157.48" y="238.76" size="1.27" layer="95" xref="yes"/>
+</segment>
+<segment>
+<pinref part="SW1" gate="G$1" pin="1"/>
+<label x="287.02" y="-20.32" size="1.27" layer="95" ratio="15" rot="R180" xref="yes"/>
+<wire x1="287.02" y1="-20.32" x2="292.1" y2="-20.32" width="0.1524" layer="91"/>
+</segment>
+</net>
+<net name="D15/SW2" class="0">
+<segment>
+<pinref part="U2" gate="G$1" pin="P0.15"/>
+<wire x1="154.94" y1="248.92" x2="157.48" y2="248.92" width="0.1524" layer="91"/>
+<label x="157.48" y="248.92" size="1.27" layer="95" xref="yes"/>
+</segment>
+<segment>
+<pinref part="SW2" gate="G$1" pin="1"/>
+<label x="320.04" y="-20.32" size="1.27" layer="95" ratio="15" rot="R180" xref="yes"/>
+<wire x1="320.04" y1="-20.32" x2="325.12" y2="-20.32" width="0.1524" layer="91"/>
+</segment>
+</net>
+<net name="D16/SW3" class="0">
+<segment>
+<pinref part="SW5" gate="G$1" pin="1"/>
+<wire x1="353.06" y1="-20.32" x2="358.14" y2="-20.32" width="0.1524" layer="91"/>
+</segment>
+</net>
+<net name="D16/CS.OLED" class="0">
+<segment>
+<pinref part="U2" gate="G$1" pin="P0.16"/>
+<wire x1="154.94" y1="251.46" x2="157.48" y2="251.46" width="0.1524" layer="91"/>
+<label x="157.48" y="251.46" size="1.27" layer="95" xref="yes"/>
+</segment>
+<segment>
+<pinref part="U3" gate="G$1" pin="/CS"/>
+<wire x1="325.12" y1="83.82" x2="322.58" y2="83.82" width="0.1524" layer="91"/>
+<label x="322.58" y="83.82" size="1.27" layer="95" rot="R180" xref="yes"/>
+<label x="322.58" y="83.82" size="1.27" layer="95" rot="R180" xref="yes"/>
+</segment>
+</net>
+<net name="D3/RESET.OLED" class="0">
+<segment>
+<pinref part="U2" gate="G$1" pin="P0.03/AIN1"/>
+<wire x1="127" y1="226.06" x2="127" y2="223.52" width="0.1524" layer="91"/>
+<label x="127" y="223.52" size="1.27" layer="95" rot="R270" xref="yes"/>
+</segment>
+<segment>
+<pinref part="U3" gate="G$1" pin="/RES"/>
+<wire x1="325.12" y1="81.28" x2="322.58" y2="81.28" width="0.1524" layer="91"/>
+<label x="322.58" y="81.28" size="1.27" layer="95" rot="R180" xref="yes"/>
+</segment>
+</net>
+<net name="D4/DC.OLED" class="0">
+<segment>
+<pinref part="U2" gate="G$1" pin="P0.04/AIN2"/>
+<wire x1="129.54" y1="226.06" x2="129.54" y2="223.52" width="0.1524" layer="91"/>
+<label x="129.54" y="223.52" size="1.27" layer="95" rot="R270" xref="yes"/>
+</segment>
+<segment>
+<pinref part="U3" gate="G$1" pin="DC/I2C_SA0"/>
+<wire x1="325.12" y1="78.74" x2="322.58" y2="78.74" width="0.1524" layer="91"/>
+<label x="322.58" y="78.74" size="1.27" layer="95" rot="R180" xref="yes"/>
+</segment>
+</net>
+<net name="D29/LED.CTRL" class="0">
+<segment>
+<pinref part="U2" gate="G$1" pin="P0.29/AIN5"/>
+<wire x1="109.22" y1="254" x2="106.68" y2="254" width="0.1524" layer="91"/>
+<label x="106.68" y="254" size="1.27" layer="95" rot="R180" xref="yes"/>
+</segment>
+</net>
+<net name="A6/TIA" class="0">
+<segment>
+<pinref part="U2" gate="G$1" pin="P0.30/AIN6"/>
+<wire x1="109.22" y1="251.46" x2="106.68" y2="251.46" width="0.1524" layer="91"/>
+<label x="106.68" y="251.46" size="1.27" layer="95" rot="R180" xref="yes"/>
+</segment>
+</net>
+<net name="A7/PPG" class="0">
+<segment>
+<pinref part="U2" gate="G$1" pin="P0.31/AIN7"/>
+<wire x1="109.22" y1="248.92" x2="106.68" y2="248.92" width="0.1524" layer="91"/>
+<label x="106.68" y="248.92" size="1.27" layer="95" rot="R180" xref="yes"/>
+</segment>
+</net>
