File: hardware/BOTTOM/RiseUpBOTTOM.sch (EAGLE design)
At the start: 31 parts, among them U1 AD5242-SO16

Commit message: Updated Bottom board from Take 2
Parts:
- added J1: (no value), LinnesLab-Connectors:CONN_07
Other:
- note added: "Pins that need to go from bottom board to top board 3.3V Ground TIA PPG SDA SCL LED.CTRL"
Changed lines of the file:
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@@
 <part name="GND2" library="LinnesLab-Symbols" deviceset="GND" device=""/>
 <part name="SUPPLY3" library="LinnesLab-Symbols" deviceset="3.3V" device=""/>
+<part name="J1" library="LinnesLab-Connectors" deviceset="CONN_07" device=""/>
 </parts>
 <sheets>
@@
 <text x="144.78" y="10.16" size="1.778" layer="97" ratio="15">I2C Address: 0x2C</text>
 <text x="210.82" y="12.7" size="1.778" layer="97" ratio="15">I2C Address: 0x2D</text>
+<text x="264.16" y="99.06" size="1.778" layer="91">Pins that need to go from bottom board to top board
+3.3V
+Ground
+TIA
+PPG
+SDA
+SCL
+LED.CTRL</text>
 </plain>
 <instances>
@@
 <attribute name="VALUE" x="27.94" y="-3.556" size="1.778" layer="96" align="bottom-center"/>
 </instance>
+<instance part="J1" gate="G$1" x="137.16" y="-20.32" smashed="yes">
+<attribute name="VALUE" x="132.08" y="-30.226" size="1.778" layer="96" font="vector"/>
+<attribute name="NAME" x="132.08" y="-7.112" size="1.778" layer="95" font="vector"/>
+</instance>
 </instances>

Commit message: Updates end of July2nd, Start Take 03
Connections:
- removed net LED.CTRL: U$4.A
- removed net PPG: C21.2, OP3G$1.OUT, U1.B2
- removed net TIA: C10.2, C15.1, OP4G$1.OUT, U1.W1
- new net A6/TIA: C10.2, C15.1, J1.5, OP4G$1.OUT, U1.W1
- new net A7/PPG: C21.2, J1.7, OP3G$1.OUT, U1.B2
- new net D29/LED.CTRL: J1.6, U$4.A
Changed lines of the file:
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@@
 <text x="144.78" y="10.16" size="1.778" layer="97" ratio="15">I2C Address: 0x2C</text>
 <text x="210.82" y="12.7" size="1.778" layer="97" ratio="15">I2C Address: 0x2D</text>
-<text x="264.16" y="99.06" size="1.778" layer="91">Pins that need to go from bottom board to top board
+<text x="264.16" y="99.06" size="1.778" layer="97">Pins that need to go from bottom board to top board
 3.3V
 Ground
@@
 </segment>
 </net>
-<net name="TIA" class="0">
+<net name="A6/TIA" class="0">
 <segment>
 <wire x1="142.24" y1="33.02" x2="137.16" y2="33.02" width="0.1524" layer="91"/>
@@
 <junction x="85.09" y="102.87"/>
 </segment>
+<segment>
+<pinref part="J1" gate="G$1" pin="5"/>
+<wire x1="142.24" y1="-15.24" x2="149.86" y2="-15.24" width="0.1524" layer="91"/>
+<label x="149.86" y="-15.24" size="1.27" layer="95" xref="yes"/>
+</segment>
 </net>
 <net name="PD.C" class="0">
@@
 </segment>
 </net>
-<net name="LED.CTRL" class="0">
+<net name="D29/LED.CTRL" class="0">
 <segment>
 <pinref part="U$4" gate="G$1" pin="A"/>
@@
 <wire x1="238.76" y1="35.56" x2="238.76" y2="43.18" width="0.1524" layer="91"/>
 <label x="238.76" y="43.18" size="1.27" layer="95" rot="R180" xref="yes"/>
+</segment>
+<segment>
+<pinref part="J1" gate="G$1" pin="6"/>
+<wire x1="142.24" y1="-12.7" x2="149.86" y2="-12.7" width="0.1524" layer="91"/>
+<label x="149.86" y="-12.7" size="1.27" layer="95" xref="yes"/>
 </segment>
 </net>
@@
 </segment>
 </net>
-<net name="PPG" class="0">
+<net name="A7/PPG" class="0">
 <segment>
 <wire x1="170.18" y1="33.02" x2="172.72" y2="33.02" width="0.1524" layer="91"/>
@@
 <label x="224.79" y="95.25" size="1.27" layer="95" xref="yes"/>
 </segment>
-</net>
+<segment>
+<pinref part="J1" gate="G$1" pin="7"/>
+<wire x1="142.24" y1="-10.16" x2="149.86" y2="-10.16" width="0.1524" layer="91"/>
+<label x="149.86" y="-10.16" size="1.27" layer="95" xref="yes"/>
+</segment>
+</net>

Commit message: Updated Bottom board Take 3
Connections:
- removed net LED: Q1.C
- net 3.3V: now also J1.4
- net GND: now also J1.3
- net LED.C: now also Q1.C
- net SCL: now also J1.2
- net SDA: now also J1.1
Changed lines of the file:
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@@
 <part name="SUPPLY3" library="LinnesLab-Symbols" deviceset="3.3V" device=""/>
 <part name="J1" library="LinnesLab-Connectors" deviceset="CONN_07" device=""/>
+<part name="GND3" library="LinnesLab-Symbols" deviceset="GND" device=""/>
+<part name="SUPPLY1" library="LinnesLab-Symbols" deviceset="3.3V" device=""/>
 </parts>
 <sheets>
@@
 <attribute name="NAME" x="132.08" y="-7.112" size="1.778" layer="95" font="vector"/>
 </instance>
+<instance part="GND3" gate="G$1" x="147.32" y="-33.02" smashed="yes">
+<attribute name="VALUE" x="147.32" y="-33.274" size="1.778" layer="96" align="top-center"/>
+</instance>
+<instance part="SUPPLY1" gate="G$1" x="147.32" y="-5.08" smashed="yes">
+<attribute name="VALUE" x="147.32" y="-2.286" size="1.778" layer="96" align="bottom-center"/>
+</instance>
 </instances>
 <busses>
@@
 <wire x1="27.94" y1="-19.05" x2="27.94" y2="-16.51" width="0.1524" layer="91"/>
 </segment>
+<segment>
+<pinref part="J1" gate="G$1" pin="3"/>
+<wire x1="142.24" y1="-20.32" x2="147.32" y2="-20.32" width="0.1524" layer="91"/>
+<pinref part="GND3" gate="G$1" pin="GND"/>
+<wire x1="147.32" y1="-20.32" x2="147.32" y2="-30.48" width="0.1524" layer="91"/>
+</segment>
 </net>
 <net name="3.3V" class="0">
@@
 <wire x1="27.94" y1="-6.35" x2="27.94" y2="-8.89" width="0.1524" layer="91"/>
 </segment>
+<segment>
+<pinref part="J1" gate="G$1" pin="4"/>
+<wire x1="142.24" y1="-17.78" x2="147.32" y2="-17.78" width="0.1524" layer="91"/>
+<pinref part="SUPPLY1" gate="G$1" pin="3.3V"/>
+<wire x1="147.32" y1="-17.78" x2="147.32" y2="-5.08" width="0.1524" layer="91"/>
+</segment>
 </net>
 <net name="SDA" class="0">
@@
 <label x="68.58" y="-11.43" size="1.27" layer="95" xref="yes"/>
 </segment>
+<segment>
+<pinref part="J1" gate="G$1" pin="1"/>
+<wire x1="142.24" y1="-25.4" x2="149.86" y2="-25.4" width="0.1524" layer="91"/>
+<label x="149.86" y="-25.4" size="1.27" layer="95" xref="yes"/>
+</segment>
 </net>
 <net name="SCL" class="0">
@@
 <wire x1="66.04" y1="-16.51" x2="68.58" y2="-16.51" width="0.1524" layer="91"/>
 <label x="68.58" y="-16.51" size="1.27" layer="95" xref="yes"/>
+</segment>
+<segment>
+<pinref part="J1" gate="G$1" pin="2"/>
+<wire x1="142.24" y1="-22.86" x2="149.86" y2="-22.86" width="0.1524" layer="91"/>
+<label x="149.86" y="-22.86" size="1.27" layer="95" xref="yes"/>
 </segment>
 </net>
@@
 <label x="39.37" y="102.87" size="1.27" layer="95" xref="yes"/>
 </segment>
+<segment>
+<wire x1="259.08" y1="35.56" x2="259.08" y2="38.1" width="0.1524" layer="91"/>
+<label x="259.08" y="38.1" size="1.27" layer="95" rot="R180" xref="yes"/>
+<pinref part="Q1" gate="G$1" pin="C"/>
+</segment>
 </net>
 <net name="VREF" class="0">
@@
 </segment>
 </net>
-<net name="LED" class="0">
-<segment>
-<wire x1="259.08" y1="35.56" x2="259.08" y2="38.1" width="0.1524" layer="91"/>
-<label x="259.08" y="38.1" size="1.27" layer="95" rot="R180" xref="yes"/>
-<pinref part="Q1" gate="G$1" pin="C"/>
-</segment>
-</net>
